File: brake-node-hat.kicad_pcb (KiCad board)
At the start: 2 copper layers, 46 x 30 mm, 19 parts, among them J1 Screw_Terminal_01x02, J4 Screw_Terminal_01x02, J5 Screw_Terminal_01x02, J6 Screw_Terminal_01x02, J7 Screw_Terminal_01x02

Commit message: adding gerber zip
Parts:
- moved J4 0.58 mm to (181.9, 109.9)
- moved CT 0.28 mm to (183.0, 94.5)
- moved J7 0.24 mm to (163.3, 91.6)
- moved R3 0.23 mm to (191.0, 90.2)
- moved J1 0.20 mm to (196.2, 112.1)
- moved R5 0.20 mm to (170.3, 101.5)
- moved R1 0.10 mm to (190.6, 101.0)
- moved R2 0.10 mm to (188.3, 100.3)
- moved RSC 0.10 mm to (196.0, 94.5)
Routing:
- net VDD: track 0.00 -> 29.4 mm
- net VD: track 0.00 -> 25.9 mm
- net +12V: track 0.00 -> 20.1 mm
- net Net-(J4-Pin_1): track 0.00 -> 12.6 mm
- net Net-(U1-I_PEAK_Sense): track 0.00 -> 12.4 mm
- net Net-(J6-Pin_1): track 0.00 -> 11.4 mm
- net Net-(D1-A): track 0.00 -> 7.71 mm
- net Net-(U1-Comparator_Inverting_Input): track 0.00 -> 4.19 mm
- net Net-(U1-Timing_Capacitor): track 0.00 -> 2.72 mm
- net Net-(U1-Driver_Collector): track 0.00 -> 2.28 mm
- net GND: vias 0 -> 69
- added copper zone on B.Cu, net GND
- added copper zone on F.Cu, net GND
